Commit message: delete the dummy link in urdf file, fixed odom not published problem

File: myhamster_simulation/urdf/hamster.urdf.xacro (robot description, xacro)
@@ -11,5 +11,5 @@
   <xacro:arg name="robot_version" default="V6"/>
   <xacro:property name="version" value="$(arg robot_version)"/>
-  <link name="dummy"/>
+  <!--link name="dummy"/-->
   <link name="base_link">
     <inertial>
@@ -39,9 +39,9 @@
     </visual>
     </link>
-  <joint name="dummy_link_joint" type="fixed">
+  <!--joint name="dummy_link_joint" type="fixed">
     <origin xyz="0 0 0" rpy="0 0 0" />
     <parent link="dummy" />
     <child  link="base_link" />
-  </joint>
+  </joint-->
   <joint name="imu_link_joint" type="fixed">
     <origin xyz="0 0 0" rpy="0 0 0" />
