Commit message: add ackermann gazebo plugin, increase maximum steering angle

File: myhamster_simulation/urdf/front_wheel.urdf.xacro (robot description, xacro)
@@ -54,5 +54,5 @@
       <mu1>0.7</mu1>
       <mu2>0.7</mu2>
-      <kp>500000.0</kp>
+      <kp>50000000.0</kp>
       <kd>10.0</kd>
       <minDepth>0.002</minDepth>
@@ -75,5 +75,5 @@
       <origin xyz="${origin_x} ${origin_y} ${origin_z}" rpy="0 0 0" />
       <axis xyz="0 0 1" rpy="0 0 0" />
-      <limit effort="30" velocity="1.5" lower="-0.296706" upper="0.296706"/>
+      <limit effort="30" velocity="1.5" lower="-0.4" upper="0.4"/>
       <!-- <dynamics damping="0.7"/> -->
     </joint>

File: myhamster_simulation/urdf/rear_wheel.urdf.xacro (robot description, xacro)
@@ -41,5 +41,5 @@
       <mu1>0.7</mu1>
       <mu2>0.7</mu2>
-      <kp>500000.0</kp>
+      <kp>50000000.0</kp>
       <kd>10.0</kd>
       <minDepth>0.002</minDepth>

Commit message: tune teb local planner parameters

File: myhamster_simulation/urdf/front_wheel.urdf.xacro (robot description, xacro)
@@ -75,5 +75,5 @@
       <origin xyz="${origin_x} ${origin_y} ${origin_z}" rpy="0 0 0" />
       <axis xyz="0 0 1" rpy="0 0 0" />
-      <limit effort="30" velocity="1.5" lower="-0.4" upper="0.4"/>
+      <limit effort="30" velocity="1.5" lower="-0.5" upper="0.5"/>
       <!-- <dynamics damping="0.7"/> -->
     </joint>

Commit message: tune wheel params and add new world file

File: myhamster_simulation/urdf/front_wheel.urdf.xacro (robot description, xacro)
@@ -4,5 +4,5 @@
   <xacro:property name="wheel_radius" value="0.029" />
   <xacro:property name="wheel_height" value="0.02" />
-  <xacro:property name="wheel_mass" value="0.1" /> <!-- in kg-->
+  <xacro:property name="wheel_mass" value="0.5" /> <!-- in kg-->
   <xacro:macro name="cylinder_inertia" params="m r h">
     <inertia  ixx="${m*(3*r*r+h*h)/12}" ixy="0" ixz="0"
@@ -54,10 +54,10 @@
       <mu1>100.0</mu1>
       <mu2>50.0</mu2>
-      <kp>1000000.0</kp>
-      <kd>10.0</kd>
-      <minDepth>0.002</minDepth>
-      <maxVel>0.1</maxVel>
+      <kp>10000000.0</kp>
+      <kd>1.0</kd>
+      <!--minDepth>0.002</minDepth-->
+      <!--maxVel>0.1</maxVel-->
       <fdir1>1 0 0</fdir1>
-      <maxContacts>20</maxContacts>
+      <!--maxContacts>20</maxContacts-->
       <!-- <material>Gazebo/FlatBlack</material> -->
     </gazebo>

File: myhamster_simulation/urdf/rear_wheel.urdf.xacro (robot description, xacro)
@@ -4,5 +4,5 @@
   <xacro:property name="wheel_radius" value="0.029" />
   <xacro:property name="wheel_height" value="0.02" />
-  <xacro:property name="wheel_mass" value="0.1" /> <!-- in kg-->
+  <xacro:property name="wheel_mass" value="0.5" /> <!-- in kg-->
   <xacro:macro name="cylinder_inertia" params="m r h">
     <inertia  ixx="${m*(3*r*r+h*h)/12}" ixy="0" ixz="0"
@@ -41,11 +41,11 @@
       <mu1>100.0</mu1>
       <mu2>50.0</mu2>
-      <kp>1000000.0</kp>
-      <kd>10.0</kd>
-      <minDepth>0.002</minDepth>
-      <maxVel>0.1</maxVel>
+      <kp>10000000.0</kp>
+      <kd>1.0</kd>
+      <!--minDepth>0.002</minDepth-->
+      <!--maxVel>0.1</maxVel-->
       <fdir1>1 0 0</fdir1>
       <!-- <material>Gazebo/FlatBlack</material> -->
-      <maxContacts>20</maxContacts>
+      <!--maxContacts>20</maxContacts-->
     </gazebo>
     <joint name="${fr}_${lr}_wheel_joint" type="continuous">

Commit message: add curve shape driving

File: myhamster_simulation/urdf/front_wheel.urdf.xacro (robot description, xacro)
@@ -61,4 +61,5 @@
       <!--maxContacts>20</maxContacts-->
       <!-- <material>Gazebo/FlatBlack</material> -->
+      <material>Gazebo/Blue</material>
     </gazebo>
     <joint name="${fr}_${lr}_wheel_joint" type="continuous">

File: myhamster_simulation/urdf/hamster.urdf.xacro (robot description, xacro)
@@ -28,4 +28,7 @@
     </collision>
   </link>
+  <gazebo reference="base_link">
+    <material>Gazebo/Green</material>
+  </gazebo>
   <link name="imu_link">
     <inertial>

File: myhamster_simulation/urdf/rear_wheel.urdf.xacro (robot description, xacro)
@@ -48,4 +48,5 @@
       <!-- <material>Gazebo/FlatBlack</material> -->
       <!--maxContacts>20</maxContacts-->
+      <material>Gazebo/Blue</material>
     </gazebo>
     <joint name="${fr}_${lr}_wheel_joint" type="continuous">
